File: corrupt_core_eagle_files/CorruptCore.sch (EAGLE design)
At the start: 90 parts, among them K1 DTS-3, K10 DTS-3, K11 DTS-3, K12 DTS-3, K13 DTS-3, K14 DTS-3, K15 DTS-3, K16 DTS-3, K2 DTS-3, K3 DTS-3, K4 DTS-3, K5 DTS-3, K6 DTS-3, K7 DTS-3, K8 DTS-3, K9 DTS-3, T1 TRANS_NPN-MMBTA42, T2 TRANS_NPN-MMBTA42, T3 TRANS_NPN-MMBTA42, T4 TRANS_NPN-MMBTA42, U1 MEGA8-P, U2 SNX4HC595SOIC16, U3 SNX4HC595SOIC16, U4 SNX4HC595SOIC16, U5 ULN2803ASOIC18, U6 ULN2803ASOIC18, U7 ULN2803ASOIC18, U8 LTC1799, Y1 16MHz

Commit message: -fixed license
Other:
- note added: "License: GNU General Public License V3"
- note removed: "License: Creative Commons Attribution-ShareAlike CC BY-SA"
Changed lines of the file:
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@@
 <text x="261.62" y="-63.5" size="1.778" layer="94">Author: Grant Haack</text>
 <text x="261.62" y="-68.58" size="1.778" layer="94">Rev: 0.4</text>
-<text x="261.62" y="-76.2" size="1.778" layer="94">License: Creative Commons Attribution-ShareAlike
-CC BY-SA</text>
+<text x="261.62" y="-73.66" size="1.778" layer="94">License: GNU General Public License V3</text>
 </plain>
 <instances>
@@
 </drawing>
 <compatibility>
-<note version="6.3" minversion="6.2.2" severity="warning">
-Since Version 6.2.2 text objects can contain more than one line,
-which will not be processed correctly with this version.
-</note>
 <note version="8.2" severity="warning">
 Since Version 8.2, Eagle supports online libraries. The ids
